File: pcb/XBee_esp8266.kicad_pcb (KiCad board)
At the start: 2 copper layers, 24.5 x 27 mm, 5 parts, among them P1 CONN_XBEE1, P3 CONN_ESP8266, P4 CONN_XBEE2, SW1 SW_CONFIG

Commit message: updated gerbers
Parts:
- removed C_SRL: CONN_SERIAL, Pin_Headers:Pin_Header_Straight_1x06
- added P2: CONN_SERIAL, Pin_Headers:Pin_Header_Straight_1x06, F.Cu at (191.2, 122.8)
- turned P3 to 180 degrees
Routing:
- net Net-(P1-Pad3): track 41.5 -> 28.2 mm, vias 1 -> 0
- net Net-(P3-Pad5): track 28.4 -> 16.0 mm
- net Net-(P2-Pad2): track 28.8 -> 22.0 mm, vias 1 -> 0
- net +3.3V: track 18.0 -> 16.5 mm
- net Net-(P2-Pad1): track 0.00 -> 1.05 mm
